Commit message: Update robot.urdf.xacro

File: workspace_tito/src/tito_controllers/urdf/robot.urdf.xacro (robot description, xacro)
@@ -4,5 +4,5 @@
   <origin xyz="0 0 0" rpy="0 0 0"/>
     <geometry>
-      <mesh filename="file:///home/fac/Desktop/robot_diff_tesis.stl"
+      <mesh "package://mi_robot_description/meshes/robot_diff_tesis.stl"
             scale="0.01 0.01 0.01"/>
     </geometry>

Commit message: Update mesh path for robot model in URDF

File: workspace_tito/src/tito_controllers/urdf/robot.urdf.xacro (robot description, xacro)
@@ -4,5 +4,5 @@
   <origin xyz="0 0 0" rpy="0 0 0"/>
     <geometry>
-      <mesh "package://mi_robot_description/meshes/robot_diff_tesis.stl"
+      <mesh "package://tito_controllers/meshes/robot_diff_tesis.stl"
             scale="0.01 0.01 0.01"/>
     </geometry>

Commit message: .

File: workspace_tito/src/tito_controllers/urdf/robot.urdf.xacro (robot description, xacro)
@@ -4,5 +4,5 @@
   <origin xyz="0 0 0" rpy="0 0 0"/>
     <geometry>
-      <mesh filename="file:///home/fac/Desktop/robot_diff_tesis.stl"
+      <mesh "package://tito_controllers/meshes/robot_diff_tesis.stl"
             scale="0.01 0.01 0.01"/>
     </geometry>
